File: elec/asserv_dc/asserv_dc.kicad_pcb (KiCad board)
At the start: 2 copper layers, 88 x 55 mm, 49 parts, among them J1 Conn_01x02, J2 Conn_01x04, J3 Conn_01x04, J4 Conn_01x02, J5 Conn_01x02, U1 Nucleo-F303K8, U2 VNH5019A-E, U3 74AHC2G00, U4 VNH5019A-E, U5 IRFR014PBF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

Commit message: V1.1 : fix current sense (CS and CS1) pins of VNH5019 not connected to uC
Connections:
- U1 pad 21: Net-(U1-Pad21) -> /CS
- U1 pad 23: Net-(U1-Pad23) -> /CS1
- U3 pad 8: +5VL -> VCC
Routing:
- net /CS: track 4.58 -> 27.6 mm, vias 0 -> 2
- net /CS1: track 4.58 -> 12.7 mm, vias 0 -> 2
Other:
- board text added: "DC Motors V1.1"
