File: elec/asserv_dc/asserv_dc.sch (KiCad schematic (older format))
At the start: 44 parts, among them J1 Conn_01x02, J2 Conn_01x04, J3 Conn_01x04, J4 Conn_01x02, J5 Conn_01x02, U1 Nucleo-F303K8, U2 VNH5019A-E, U3 74AHC2G00, U4 VNH5019A-E, U5 IRFR014PBF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

Commit message: V1.1 : fix current sense (CS and CS1) pins of VNH5019 not connected to uC
Connections:
- net CS: now also U1.21 (PA_3)
- net CS1: now also U1.23 (PA_5)
Changed lines of the file:
@@
 Wire Wire Line
 	3100 1700 3100 1800
+Text Label 3450 4150 0    50   ~ 0
+CS
+Wire Wire Line
+	3450 4150 3350 4150
+Text Label 3450 4350 0    50   ~ 0
+CS1
+Wire Wire Line
+	3450 4350 3350 4350
 $EndSCHEMATC
